Commit message: added 4 intermediate spaces for the blocks

File: cu_panda_description/robots/basic_setup.urdf.xacro (robot description, xacro)
@@ -48,4 +48,64 @@
     </collision>
   </link>
+  <link name="intermediate_space_1">
+    <visual>
+      <geometry>
+        <box size="0.07 0.07 0.05"/>
+      </geometry>
+      <material name="orange">
+        <color rgba="1.0 0.5 0.0 0.5"/>
+      </material>
+    </visual>
+  </link>
+  <joint name="intermediate_space_joint_1" type="fixed">
+    <child link="intermediate_space_1"/>
+    <parent link="table_top"/>
+    <origin xyz="0.2 -0.035 0" rpy="0 0 0"/>
+  </joint>
+    <link name="intermediate_space_2">
+    <visual>
+      <geometry>
+        <box size="0.07 0.07 0.05"/>
+      </geometry>
+      <material name="orange">
+        <color rgba="1.0 0.5 0.0 0.5"/>
+      </material>
+    </visual>
+  </link>
+  <joint name="intermediate_space_joint_2" type="fixed">
+    <child link="intermediate_space_2"/>
+    <parent link="table_top"/>
+    <origin xyz="0.2 0.035 0" rpy="0 0 0"/>
+  </joint>
+  <link name="intermediate_space_3">
+    <visual>
+      <geometry>
+        <box size="0.07 0.07 0.05"/>
+      </geometry>
+      <material name="orange">
+        <color rgba="1.0 0.5 0.0 0.5"/>
+      </material>
+    </visual>
+  </link>
+  <joint name="intermediate_space_joint_3" type="fixed">
+    <child link="intermediate_space_3"/>
+    <parent link="table_top"/>
+    <origin xyz="0.27 -0.035 0" rpy="0 0 0"/>
+  </joint>
+  <link name="intermediate_space_4">
+    <visual>
+      <geometry>
+        <box size="0.07 0.07 0.05"/>
+      </geometry>
+      <material name="orange">
+        <color rgba="1.0 0.5 0.0 0.5"/>
+      </material>
+    </visual>
+  </link>
+  <joint name="intermediate_space_joint_4" type="fixed">
+    <child link="intermediate_space_4"/>
+    <parent link="table_top"/>
+    <origin xyz="0.27 0.035 0" rpy="0 0 0"/>
+  </joint>
   <joint name="mounting_table_joint" type="fixed">
     <child link="panda_mounting_plate"/>

Commit message: chnaged rviz config and changed pos of ittermediate areas to avoid collisions due to errors

File: cu_panda_description/robots/basic_setup.urdf.xacro (robot description, xacro)
@@ -61,5 +61,5 @@
     <child link="intermediate_space_1"/>
     <parent link="table_top"/>
-    <origin xyz="0.2 -0.035 0" rpy="0 0 0"/>
+    <origin xyz="0.17 -0.037 0" rpy="0 0 0"/>
   </joint>
     <link name="intermediate_space_2">
@@ -76,5 +76,5 @@
     <child link="intermediate_space_2"/>
     <parent link="table_top"/>
-    <origin xyz="0.2 0.035 0" rpy="0 0 0"/>
+    <origin xyz="0.17 0.037 0" rpy="0 0 0"/>
   </joint>
   <link name="intermediate_space_3">
@@ -91,5 +91,5 @@
     <child link="intermediate_space_3"/>
     <parent link="table_top"/>
-    <origin xyz="0.27 -0.035 0" rpy="0 0 0"/>
+    <origin xyz="0.25 -0.037 0" rpy="0 0 0"/>
   </joint>
   <link name="intermediate_space_4">
@@ -106,5 +106,5 @@
     <child link="intermediate_space_4"/>
     <parent link="table_top"/>
-    <origin xyz="0.27 0.035 0" rpy="0 0 0"/>
+    <origin xyz="0.25 0.037 0" rpy="0 0 0"/>
   </joint>
   <joint name="mounting_table_joint" type="fixed">

Commit message: changed pos of intermediate spaces for better reachability

File: cu_panda_description/robots/basic_setup.urdf.xacro (robot description, xacro)
@@ -61,5 +61,5 @@
     <child link="intermediate_space_1"/>
     <parent link="table_top"/>
-    <origin xyz="0.17 -0.037 0" rpy="0 0 0"/>
+    <origin xyz="0.16 -0.038 0" rpy="0 0 0"/>
   </joint>
     <link name="intermediate_space_2">
@@ -76,5 +76,5 @@
     <child link="intermediate_space_2"/>
     <parent link="table_top"/>
-    <origin xyz="0.17 0.037 0" rpy="0 0 0"/>
+    <origin xyz="0.16 0.038 0" rpy="0 0 0"/>
   </joint>
   <link name="intermediate_space_3">
@@ -91,5 +91,5 @@
     <child link="intermediate_space_3"/>
     <parent link="table_top"/>
-    <origin xyz="0.25 -0.037 0" rpy="0 0 0"/>
+    <origin xyz="0.24 -0.038 0" rpy="0 0 0"/>
   </joint>
   <link name="intermediate_space_4">
@@ -106,5 +106,5 @@
     <child link="intermediate_space_4"/>
     <parent link="table_top"/>
-    <origin xyz="0.25 0.037 0" rpy="0 0 0"/>
+    <origin xyz="0.24 0.038 0" rpy="0 0 0"/>
   </joint>
   <joint name="mounting_table_joint" type="fixed">

Commit message: changed location of intermediate spaces

File: cu_panda_description/robots/basic_setup.urdf.xacro (robot description, xacro)
@@ -61,5 +61,5 @@
     <child link="intermediate_space_1"/>
     <parent link="table_top"/>
-    <origin xyz="0.16 -0.038 0" rpy="0 0 0"/>
+    <origin xyz="0.15 -0.175 0" rpy="0 0 0"/>
   </joint>
     <link name="intermediate_space_2">
@@ -76,5 +76,5 @@
     <child link="intermediate_space_2"/>
     <parent link="table_top"/>
-    <origin xyz="0.16 0.038 0" rpy="0 0 0"/>
+    <origin xyz="0.15 -0.10 0" rpy="0 0 0"/>
   </joint>
   <link name="intermediate_space_3">
@@ -91,5 +91,5 @@
     <child link="intermediate_space_3"/>
     <parent link="table_top"/>
-    <origin xyz="0.24 -0.038 0" rpy="0 0 0"/>
+    <origin xyz="0.15 -0.025 0" rpy="0 0 0"/>
   </joint>
   <link name="intermediate_space_4">
@@ -99,5 +99,5 @@
       </geometry>
       <material name="orange">
-        <color rgba="1.0 0.5 0.0 0.5"/>
+        <color rgba="1.0 0.6 0.0 0.5"/>
       </material>
     </visual>
@@ -106,5 +106,5 @@
     <child link="intermediate_space_4"/>
     <parent link="table_top"/>
-    <origin xyz="0.24 0.038 0" rpy="0 0 0"/>
+    <origin xyz="0.15 0.05 0" rpy="0 0 0"/>
   </joint>
   <joint name="mounting_table_joint" type="fixed">

Commit message: recalibrated camera

File: cu_panda_description/robots/basic_setup.urdf.xacro (robot description, xacro)
@@ -61,5 +61,5 @@
     <child link="intermediate_space_1"/>
     <parent link="table_top"/>
-    <origin xyz="0.15 -0.175 0" rpy="0 0 0"/>
+    <origin xyz="0.17 -0.175 0" rpy="0 0 0"/>
   </joint>
     <link name="intermediate_space_2">
@@ -76,5 +76,5 @@
     <child link="intermediate_space_2"/>
     <parent link="table_top"/>
-    <origin xyz="0.15 -0.10 0" rpy="0 0 0"/>
+    <origin xyz="0.17 -0.10 0" rpy="0 0 0"/>
   </joint>
   <link name="intermediate_space_3">
@@ -91,5 +91,5 @@
     <child link="intermediate_space_3"/>
     <parent link="table_top"/>
-    <origin xyz="0.15 -0.025 0" rpy="0 0 0"/>
+    <origin xyz="0.17 -0.025 0" rpy="0 0 0"/>
   </joint>
   <link name="intermediate_space_4">
@@ -106,10 +106,10 @@
     <child link="intermediate_space_4"/>
     <parent link="table_top"/>
-    <origin xyz="0.15 0.05 0" rpy="0 0 0"/>
+    <origin xyz="0.17 0.05 0" rpy="0 0 0"/>
   </joint>
   <joint name="mounting_table_joint" type="fixed">
     <child link="panda_mounting_plate"/>
     <parent link="table"/>
-    <origin xyz="${-0.35+0.16} ${-0.537+0.04+0.108} 0.026" rpy="0 0 0"/>
+    <origin xyz="${-0.35+0.16} ${-0.537+0.04+0.108} 0.027" rpy="0 0 0"/>
   </joint>
   <link name="table_top"/>
@@ -117,5 +117,5 @@
     <child link="table_top"/>
     <parent link="table"/>
-    <origin xyz="0 0 0.026" rpy="0 0 0"/>
+    <origin xyz="0 0 0.027" rpy="0 0 0"/>
   </joint>
   <link name="window_collider">
@@ -181,4 +181,5 @@
     <origin xyz="${-0.35-0.095} 0 ${0.026}" rpy="0 0 0"/>
   </joint>
+ <!-- # -0.353; 0.48923; 0.3458 -->
   <link name="realsense_link">
     <collision>
@@ -192,5 +193,5 @@
     <child link="realsense_link"/>
     <parent link="table"/>
-    <origin xyz="-0.34866 0.48523 0.34558" rpy="-2.9583 2.6983 2.2201"/>
+    <origin xyz="-0.360 0.490 0.342" rpy="0.192 0.436 -0.908"/>
   </joint>
   <xacro:macro name="fingertip" params="side *origin">

Commit message: fixed camera calibration, again

File: cu_panda_description/robots/basic_setup.urdf.xacro (robot description, xacro)
@@ -193,5 +193,5 @@
     <child link="realsense_link"/>
     <parent link="table"/>
-    <origin xyz="-0.360 0.490 0.342" rpy="0.192 0.436 -0.908"/>
+    <origin xyz="-0.359 0.488 0.344" rpy="0.192 0.436 -0.908"/>
   </joint>
   <xacro:macro name="fingertip" params="side *origin">

Commit message: better calibration

File: cu_panda_description/robots/basic_setup.urdf.xacro (robot description, xacro)
@@ -193,5 +193,5 @@
     <child link="realsense_link"/>
     <parent link="table"/>
-    <origin xyz="-0.359 0.488 0.344" rpy="0.192 0.436 -0.908"/>
+    <origin xyz="-0.368 0.490 0.340" rpy="0.194 0.426 -0.899"/>
   </joint>
   <xacro:macro name="fingertip" params="side *origin">

Commit message: better calibration

File: cu_panda_description/robots/basic_setup.urdf.xacro (robot description, xacro)
@@ -132,5 +132,5 @@
     <child link="realsense_link"/>
     <parent link="table"/>
-    <origin xyz="-0.34866 0.48523 0.34558" rpy="-2.9583 2.6983 2.2201"/>
+    <origin xyz="-0.368 0.490 0.340" rpy="0.194 0.426 -0.899"/>
   </joint>
   <xacro:macro name="fingertip" params="side *origin">
